File: 02 - ELECTRONIQUE/02 - CARTE PRINCIPALE/V01/MAIN_BOARD_01.brd (EAGLE design)
At the start: 100 x 80 mm, 46 parts

Commit message: Clean up repo
Changed lines of the file:
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@@
 <attribute name="NAME" x="27.94" y="36.83" size="1.27" layer="21" rot="R270"/>
 </element>
-<element name="U$4" library="OPENBOT" library_urn="urn:adsk.eagle:library:760642" package="NSK396-2C" package3d_urn="urn:adsk.eagle:package:1585093/1" value="CONN_02_PUI" x="8.89" y="39.37" smashed="yes" rot="R90"/>
+<element name="U$4" library="OPENBOT" library_urn="urn:adsk.eagle:library:760642" package="NSK396-2C" package3d_urn="urn:adsk.eagle:package:1585093/2" value="CONN_02_PUI" x="8.89" y="39.37" smashed="yes" rot="R90"/>
 <element name="C9" library="rcl" library_urn="urn:adsk.eagle:library:334" package="E5-10,5" package3d_urn="urn:adsk.eagle:package:23372/1" value="100uF" x="7.62" y="29.718" smashed="yes" rot="R90">
 <attribute name="NAME" x="4.8768" y="34.417" size="1.27" layer="25" ratio="10" rot="R90"/>
