File: 02 - ELECTRONIQUE/03 - CARTE MOTEUR/PCB_MOTEUR_V0_1b.brd (EAGLE design)
At the start: 45 x 60 mm, 10 parts

Commit message: update
Parts:
- added J1: (no value), OPENBOT:1X02
Connections:
- net RESET: now also J1.1
- net SLEEP: now also J1.2
Routing:
- net RESET: track 0.00 -> 51.7 mm
- net SLEEP: track 44.1 -> 57.1 mm
- net STEP_L: track 16.9 -> 14.0 mm
Other:
- board text added: "CC-BY-NC-SA"
- board text added: "GND"
- board text added: "Les Karibous - 2019"
- board text added: "M3"
- board text added: "Reset"
- board text added: "Sleep"
- board text added: "VMot"
Changed lines of the file:
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@@
 <drawing>
 <settings>
-<setting alwaysvectorfont="yes"/>
+<setting alwaysvectorfont="no"/>
 <setting verticaltext="up"/>
 </settings>
@@
 <layers>
 <layer number="1" name="Top" color="4" fill="1" visible="yes" active="yes"/>
+<layer number="2" name="Route2" color="1" fill="3" visible="no" active="yes"/>
+<layer number="3" name="Route3" color="4" fill="3" visible="no" active="yes"/>
+<layer number="4" name="Route4" color="1" fill="4" visible="no" active="yes"/>
+<layer number="5" name="Route5" color="4" fill="4" visible="no" active="yes"/>
+<layer number="6" name="Route6" color="1" fill="8" visible="no" active="yes"/>
+<layer number="7" name="Route7" color="4" fill="8" visible="no" active="yes"/>
+<layer number="8" name="Route8" color="1" fill="2" visible="no" active="yes"/>
+<layer number="9" name="Route9" color="4" fill="2" visible="no" active="yes"/>
+<layer number="10" name="Route10" color="1" fill="7" visible="no" active="yes"/>
+<layer number="11" name="Route11" color="4" fill="7" visible="no" active="yes"/>
+<layer number="12" name="Route12" color="1" fill="5" visible="no" active="yes"/>
+<layer number="13" name="Route13" color="4" fill="5" visible="no" active="yes"/>
+<layer number="14" name="Route14" color="1" fill="6" visible="no" active="yes"/>
+<layer number="15" name="Route15" color="4" fill="6" visible="no" active="yes"/>
 <layer number="16" name="Bottom" color="1" fill="1" visible="yes" active="yes"/>
 <layer number="17" name="Pads" color="2" fill="1" visible="yes" active="yes"/>
@@
 <wire x1="0" y1="5" x2="5" y2="0" width="0.254" layer="20" curve="90"/>
 <wire x1="5" y1="0" x2="40" y2="0" width="0.254" layer="20"/>
+<text x="24.765" y="57.15" size="1.27" layer="25" ratio="3">Sleep</text>
+<text x="13.335" y="57.15" size="1.27" layer="25" ratio="3">Reset</text>
+<text x="29.845" y="8.255" size="1.778" layer="25" ratio="3">VMot</text>
+<text x="13.335" y="5.08" size="1.27" layer="25" ratio="3">Les Karibous - 2019</text>
+<text x="15.875" y="3.175" size="1.27" layer="25" ratio="3">CC-BY-NC-SA</text>
+<text x="6.985" y="57.15" size="1.27" layer="25" ratio="3">M3</text>
+<text x="29.845" y="17.78" size="1.778" layer="25" ratio="29">GND</text>
 </plain>
 <attributes>
@@
 <element name="U$1" library="KARIBOUS" library_urn="urn:adsk.eagle:library:1283574" package="DRIVER_CARRIER_POLOLU_16" package3d_urn="urn:adsk.eagle:package:1283583/2" value="" x="27.305" y="36.83" smashed="yes" rot="R180"/>
 <element name="U$2" library="KARIBOUS" library_urn="urn:adsk.eagle:library:1283574" package="DRIVER_CARRIER_POLOLU_16" package3d_urn="urn:adsk.eagle:package:1283583/2" value="" x="27.305" y="13.97" smashed="yes" rot="R180"/>
+<element name="J1" library="OPENBOT" library_urn="urn:adsk.eagle:library:760642" package="1X02" package3d_urn="urn:adsk.eagle:package:777848/4" value="" x="19.685" y="57.785" smashed="yes">
+<attribute name="NAME" x="17.78" y="59.182" size="0.6096" layer="25" font="vector" ratio="20"/>
+<attribute name="VALUE" x="18.415" y="55.753" size="0.6096" layer="27" font="vector" ratio="20"/>
+</element>
 </elements>
 <signals>
@@
 <contactref element="J4" pad="1"/>
 <wire x1="27.305" y1="52.07" x2="28.575" y2="52.07" width="0.6096" layer="1"/>
-<wire x1="28.575" y1="52.07" x2="31.115" y2="49.53" width="0.6096" layer="1"/>
-<wire x1="31.115" y1="49.53" x2="31.115" y2="43.815" width="0.6096" layer="1"/>
-<wire x1="36.195" y1="43.815" x2="36.195" y2="42.545" width="0.6096" layer="1"/>
-<wire x1="36.195" y1="43.815" x2="31.115" y2="43.815" width="0.6096" layer="1"/>
+<wire x1="28.575" y1="52.07" x2="36.195" y2="44.45" width="0.6096" layer="1"/>
+<wire x1="36.195" y1="44.45" x2="36.195" y2="42.545" width="0.6096" layer="1"/>
 </signal>
 <signal name="DIR_L">
@@
 <contactref element="U$1" pad="P$5"/>
 <contactref element="U$2" pad="P$5"/>
-<wire x1="27.305" y1="24.13" x2="27.305" y2="46.99" width="0" layer="19" extent="1-1"/>
+<contactref element="J1" pad="1"/>
+<wire x1="27.305" y1="24.13" x2="22.225" y2="24.13" width="0.6096" layer="16"/>
+<wire x1="22.225" y1="24.13" x2="20.955" y2="25.4" width="0.6096" layer="16"/>
+<wire x1="20.955" y1="25.4" x2="20.955" y2="45.72" width="0.6096" layer="16"/>
+<wire x1="20.955" y1="45.72" x2="22.225" y2="46.99" width="0.6096" layer="16"/>
+<wire x1="22.225" y1="46.99" x2="27.305" y2="46.99" width="0.6096" layer="16"/>
+<wire x1="20.955" y1="46.99" x2="19.685" y2="48.26" width="0.6096" layer="1"/>
+<wire x1="19.685" y1="48.26" x2="19.685" y2="57.785" width="0.6096" layer="1"/>
+<wire x1="27.305" y1="46.99" x2="20.955" y2="46.99" width="0.6096" layer="1"/>
 </signal>
 <signal name="SLEEP">
@@
 <wire x1="28.575" y1="49.53" x2="27.305" y2="49.53" width="0.6096" layer="1"/>
 <wire x1="36.195" y1="40.005" x2="29.845" y2="40.005" width="0.6096" layer="1"/>
+<contactref element="J1" pad="2"/>
+<wire x1="27.305" y1="49.53" x2="22.86" y2="49.53" width="0.6096" layer="1"/>
+<wire x1="22.86" y1="49.53" x2="22.225" y2="50.165" width="0.6096" layer="1"/>
+<wire x1="22.225" y1="50.165" x2="22.225" y2="57.785" width="0.6096" layer="1"/>
 </signal>
 </signals>

Commit message: Clean up repo
Changed lines of the file:
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@@
 <attribute name="VALUE" x="36.195" y="26.416" size="0.6096" layer="27" font="vector" ratio="20" rot="R180" align="top-center"/>
 </element>
-<element name="J2" library="OPENBOT" library_urn="urn:adsk.eagle:library:760642" package="NSK396-2C" package3d_urn="urn:adsk.eagle:package:1585093/1" value="" x="32.385" y="13.97" smashed="yes" rot="R270"/>
+<element name="J2" library="OPENBOT" library_urn="urn:adsk.eagle:library:760642" package="NSK396-2C" package3d_urn="urn:adsk.eagle:package:1585093/2" value="" x="32.385" y="13.97" smashed="yes" rot="R270"/>
 <element name="J3" library="OPENBOT" library_urn="urn:adsk.eagle:library:760642" package="MOLEX-1X4" package3d_urn="urn:adsk.eagle:package:777852/5" value="" x="8.255" y="43.18" smashed="yes" rot="R90">
 <attribute name="NAME" x="4.953" y="45.466" size="0.6096" layer="25" font="vector" ratio="20" rot="R90"/>
