File: 02 - ELECTRONIQUE/03 - CARTE MOTEUR/PCB_MOTEUR_V0_1b.sch (EAGLE design)
At the start: 10 parts

Commit message: update
Parts:
- added J1: (no value), OPENBOT:CONN_02
Connections:
- net RESET: now also J1.1
- net SLEEP: now also J1.2
Changed lines of the file:
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@@
 <?xml version="1.0" encoding="utf-8"?>
 <!DOCTYPE eagle SYSTEM "eagle.dtd">
-<eagle version="9.0.0">
+<eagle version="9.2.2">
 <drawing>
 <settings>
@@
 <part name="P+9" library="supply1" library_urn="urn:adsk.eagle:library:371" deviceset="VCC" device=""/>
 <part name="GND13" library="supply1" library_urn="urn:adsk.eagle:library:371" deviceset="GNDA" device=""/>
+<part name="J1" library="OPENBOT" library_urn="urn:adsk.eagle:library:760642" deviceset="CONN_02" device="" package3d_urn="urn:adsk.eagle:package:777848/4"/>
 </parts>
 <sheets>
@@
 </plain>
 <instances>
-<instance part="U$1" gate="G$1" x="53.34" y="55.88"/>
-<instance part="J2" gate="G$1" x="-7.62" y="25.4"/>
-<instance part="J3" gate="G$1" x="88.9" y="45.72" rot="R180"/>
-<instance part="J4" gate="G$1" x="66.04" y="71.12" rot="R180"/>
-<instance part="D1" gate="G$1" x="10.16" y="53.34"/>
-<instance part="R1" gate="G$1" x="10.16" y="63.5" rot="R90"/>
-<instance part="P+2" gate="VCC" x="10.16" y="33.02"/>
-<instance part="C1" gate="G$1" x="-5.08" y="66.04"/>
-<instance part="GND2" gate="1" x="99.06" y="45.72"/>
-<instance part="GND3" gate="1" x="10.16" y="20.32"/>
-<instance part="P+3" gate="VCC" x="99.06" y="58.42"/>
-<instance part="P+4" gate="VCC" x="-5.08" y="73.66"/>
-<instance part="GND4" gate="1" x="-5.08" y="40.64"/>
-<instance part="GND5" gate="1" x="10.16" y="40.64"/>
-<instance part="P+6" gate="VCC" x="10.16" y="73.66"/>
-<instance part="GND7" gate="1" x="45.72" y="66.04"/>
-<instance part="GND8" gate="1" x="86.36" y="66.04"/>
-<instance part="GND9" gate="1" x="81.28" y="30.48"/>
-<instance part="U$2" gate="G$1" x="53.34" y="25.4"/>
-<instance part="J5" gate="G$1" x="88.9" y="15.24" rot="R180"/>
-<instance part="GND11" gate="1" x="99.06" y="15.24"/>
-<instance part="P+8" gate="VCC" x="99.06" y="27.94"/>
-<instance part="GND12" gate="1" x="81.28" y="0"/>
-<instance part="C2" gate="G$1" x="2.54" y="66.04"/>
-<instance part="P+9" gate="VCC" x="2.54" y="73.66"/>
-<instance part="GND13" gate="1" x="2.54" y="40.64"/>
+<instance part="U$1" gate="G$1" x="53.34" y="55.88" smashed="yes"/>
+<instance part="J2" gate="G$1" x="-7.62" y="25.4" smashed="yes"/>
+<instance part="J3" gate="G$1" x="88.9" y="45.72" smashed="yes" rot="R180"/>
+<instance part="J4" gate="G$1" x="66.04" y="71.12" smashed="yes" rot="R180">
+<attribute name="VALUE" x="69.85" y="81.026" size="1.778" layer="96" font="vector" rot="R180"/>
+<attribute name="NAME" x="69.85" y="62.992" size="1.778" layer="95" font="vector" rot="R180"/>
+</instance>
+<instance part="D1" gate="G$1" x="10.16" y="53.34" smashed="yes">
+<attribute name="NAME" x="6.731" y="48.768" size="1.778" layer="95" font="vector" rot="R90"/>
+<attribute name="VALUE" x="12.065" y="48.768" size="1.778" layer="96" font="vector" rot="R90" align="top-left"/>
+</instance>
+<instance part="R1" gate="G$1" x="10.16" y="63.5" smashed="yes" rot="R90">
+<attribute name="NAME" x="8.6614" y="59.69" size="1.778" layer="95" rot="R90"/>
+<attribute name="VALUE" x="13.462" y="59.69" size="1.778" layer="96" rot="R90"/>
+</instance>
+<instance part="P+2" gate="VCC" x="10.16" y="33.02" smashed="yes">
+<attribute name="VALUE" x="7.62" y="30.48" size="1.778" layer="96" rot="R90"/>
+</instance>
+<instance part="C1" gate="G$1" x="-5.08" y="66.04" smashed="yes">
+<attribute name="NAME" x="-3.937" y="66.5226" size="1.778" layer="95"/>
+<attribute name="VALUE" x="-3.937" y="61.4426" size="1.778" layer="96"/>
+</instance>
+<instance part="GND2" gate="1" x="99.06" y="45.72" smashed="yes">
+<attribute name="VALUE" x="96.52" y="43.18" size="1.778" layer="96" rot="R90"/>
+</instance>
+<instance part="GND3" gate="1" x="10.16" y="20.32" smashed="yes">
+<attribute name="VALUE" x="7.62" y="17.78" size="1.778" layer="96" rot="R90"/>
+</instance>
+<instance part="P+3" gate="VCC" x="99.06" y="58.42" smashed="yes">
+<attribute name="VALUE" x="96.52" y="55.88" size="1.778" layer="96" rot="R90"/>
+</instance>
+<instance part="P+4" gate="VCC" x="-5.08" y="73.66" smashed="yes">
+<attribute name="VALUE" x="-7.62" y="71.12" size="1.778" layer="96" rot="R90"/>
+</instance>
+<instance part="GND4" gate="1" x="-5.08" y="40.64" smashed="yes">
+<attribute name="VALUE" x="-7.62" y="38.1" size="1.778" layer="96" rot="R90"/>
+</instance>
+<instance part="GND5" gate="1" x="10.16" y="40.64" smashed="yes">
+<attribute name="VALUE" x="7.62" y="38.1" size="1.778" layer="96" rot="R90"/>
+</instance>
+<instance part="P+6" gate="VCC" x="10.16" y="73.66" smashed="yes">
+<attribute name="VALUE" x="7.62" y="71.12" size="1.778" layer="96" rot="R90"/>
+</instance>
+<instance part="GND7" gate="1" x="45.72" y="66.04" smashed="yes">
+<attribute name="VALUE" x="43.18" y="63.5" size="1.778" layer="96"/>
+</instance>
+<instance part="GND8" gate="1" x="86.36" y="66.04" smashed="yes">
+<attribute name="VALUE" x="83.82" y="63.5" size="1.778" layer="96"/>
+</instance>
+<instance part="GND9" gate="1" x="81.28" y="30.48" smashed="yes">
+<attribute name="VALUE" x="78.74" y="27.94" size="1.778" layer="96"/>
+</instance>
+<instance part="U$2" gate="G$1" x="53.34" y="25.4" smashed="yes"/>
+<instance part="J5" gate="G$1" x="88.9" y="15.24" smashed="yes" rot="R180"/>
+<instance part="GND11" gate="1" x="99.06" y="15.24" smashed="yes">
+<attribute name="VALUE" x="96.52" y="12.7" size="1.778" layer="96" rot="R90"/>
+</instance>
+<instance part="P+8" gate="VCC" x="99.06" y="27.94" smashed="yes">
+<attribute name="VALUE" x="96.52" y="25.4" size="1.778" layer="96" rot="R90"/>
+</instance>
+<instance part="GND12" gate="1" x="81.28" y="0" smashed="yes">
+<attribute name="VALUE" x="78.74" y="-2.54" size="1.778" layer="96"/>
+</instance>
+<instance part="C2" gate="G$1" x="2.54" y="66.04" smashed="yes">
+<attribute name="NAME" x="3.683" y="66.5226" size="1.778" layer="95"/>
+<attribute name="VALUE" x="3.683" y="61.4426" size="1.778" layer="96"/>
+</instance>
+<instance part="P+9" gate="VCC" x="2.54" y="73.66" smashed="yes">
+<attribute name="VALUE" x="0" y="71.12" size="1.778" layer="96" rot="R90"/>
+</instance>
+<instance part="GND13" gate="1" x="2.54" y="40.64" smashed="yes">
+<attribute name="VALUE" x="0" y="38.1" size="1.778" layer="96" rot="R90"/>
+</instance>
+<instance part="J1" gate="G$1" x="-7.62" y="10.16" smashed="yes">
+<attribute name="VALUE" x="-10.16" y="5.334" size="1.778" layer="96" font="vector"/>
+<attribute name="NAME" x="-10.16" y="15.748" size="1.778" layer="95" font="vector"/>
+</instance>
 </instances>
 <busses>
@@
 <label x="38.1" y="12.7" size="1.778" layer="95"/>
 </segment>
+<segment>
+<pinref part="J1" gate="G$1" pin="1"/>
+<wire x1="0" y1="10.16" x2="15.24" y2="10.16" width="0.1524" layer="91"/>
+<label x="12.7" y="10.16" size="1.778" layer="95"/>
+</segment>
 </net>
 <net name="SLEEP" class="0">
@@
 <label x="73.66" y="68.58" size="1.778" layer="95"/>
 </segment>
-</net>
+<segment>
+<pinref part="J1" gate="G$1" pin="2"/>
+<wire x1="0" y1="12.7" x2="10.16" y2="12.7" width="0.1524" layer="91"/>
+<label x="10.16" y="12.7" size="1.778" layer="95"/>
+</segment>
+</net>
