File: 02 - ELECTRONIQUE/04 - CARTE E-STOP/CARTE E-STOP.brd (EAGLE design)
At the start: 44 x 69.5 mm, 17 parts, among them K2 CB1-P-24V

Commit message: Clean up repo
Parts:
- added U$2: CONN_02_PUI, OPENBOT:NSK396-2C
- moved D1 1.27 mm to (27.9, 53.3)
- moved D3 1.27 mm to (20.3, 53.3)
- moved J1 1.27 mm to (27.9, 64.8)
- moved J3 1.27 mm to (20.3, 64.8)
- moved R1 1.27 mm to (30.5, 58.4)
- moved R3 1.27 mm to (22.9, 58.4)
Connections:
- net BAU: now also U$2.P$1
- net GND: now also U$2.P$2
Routing:
- net BAU: track 6.39 -> 25.1 mm
- net +24V: track 15.1 -> 13.8 mm
