File: 02 - ELECTRONIQUE/04 - CARTE E-STOP/CARTE E-STOP.sch (EAGLE design)
At the start: 17 parts, among them K2 CB1-P-24V

Commit message: Clean up repo
Parts:
- added U$2: CONN_02_PUI, OPENBOT:CONN_02_PUI
Connections:
- net BAU: now also U$2.GND/COM
- net GND: now also U$2.V+/VCC
Changed lines of the file:
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@@
 <part name="R2" library="rcl" library_urn="urn:adsk.eagle:library:334" deviceset="R-EU_" device="0207/2V" package3d_urn="urn:adsk.eagle:package:23490/1"/>
 <part name="R3" library="rcl" library_urn="urn:adsk.eagle:library:334" deviceset="R-EU_" device="0207/2V" package3d_urn="urn:adsk.eagle:package:23490/1"/>
-<part name="U$3" library="OPENBOT" library_urn="urn:adsk.eagle:library:760642" deviceset="CONN_02_PUI" device="" package3d_urn="urn:adsk.eagle:package:1585093/1"/>
-<part name="U$4" library="OPENBOT" library_urn="urn:adsk.eagle:library:760642" deviceset="CONN_02_PUI" device="" package3d_urn="urn:adsk.eagle:package:1585093/1"/>
+<part name="U$3" library="OPENBOT" library_urn="urn:adsk.eagle:library:760642" deviceset="CONN_02_PUI" device="" package3d_urn="urn:adsk.eagle:package:1585093/2"/>
+<part name="U$4" library="OPENBOT" library_urn="urn:adsk.eagle:library:760642" deviceset="CONN_02_PUI" device="" package3d_urn="urn:adsk.eagle:package:1585093/2"/>
 <part name="GND5" library="supply1" library_urn="urn:adsk.eagle:library:371" deviceset="GND" device=""/>
 <part name="GND6" library="supply1" library_urn="urn:adsk.eagle:library:371" deviceset="GND" device=""/>
@@
 <part name="BATTERIE1" library="supply2" library_urn="urn:adsk.eagle:library:372" deviceset="+24V" device=""/>
 <part name="BATTERIE2" library="supply2" library_urn="urn:adsk.eagle:library:372" deviceset="+24V" device=""/>
-<part name="U$5" library="OPENBOT" library_urn="urn:adsk.eagle:library:760642" deviceset="CONN_02_PUI" device="" package3d_urn="urn:adsk.eagle:package:1585093/1"/>
+<part name="U$5" library="OPENBOT" library_urn="urn:adsk.eagle:library:760642" deviceset="CONN_02_PUI" device="" package3d_urn="urn:adsk.eagle:package:1585093/2"/>
 <part name="GND10" library="supply1" library_urn="urn:adsk.eagle:library:371" deviceset="GND" device=""/>
 <part name="BATTERIE3" library="supply2" library_urn="urn:adsk.eagle:library:372" deviceset="+24V" device=""/>
@@
 <part name="BATTERIE6" library="supply2" library_urn="urn:adsk.eagle:library:372" deviceset="+24V" device=""/>
 <part name="D4" library="diode" library_urn="urn:adsk.eagle:library:210" deviceset="1N4004" device="" package3d_urn="urn:adsk.eagle:package:43336/1" value="1N4007"/>
-<part name="U$1" library="OPENBOT" library_urn="urn:adsk.eagle:library:760642" deviceset="CONN_02_PUI" device="" package3d_urn="urn:adsk.eagle:package:1585093/1"/>
+<part name="U$1" library="OPENBOT" library_urn="urn:adsk.eagle:library:760642" deviceset="CONN_02_PUI" device="" package3d_urn="urn:adsk.eagle:package:1585093/2"/>
 <part name="GND12" library="supply1" library_urn="urn:adsk.eagle:library:371" deviceset="GND" device=""/>
 <part name="BATTERIE5" library="supply2" library_urn="urn:adsk.eagle:library:372" deviceset="+24V" device=""/>
+<part name="U$2" library="OPENBOT" library_urn="urn:adsk.eagle:library:760642" deviceset="CONN_02_PUI" device="" package3d_urn="urn:adsk.eagle:package:1585093/2"/>
 </parts>
 <sheets>
@@
 <attribute name="VALUE" x="66.675" y="35.56" size="1.778" layer="96" rot="R270"/>
 </instance>
+<instance part="U$2" gate="G$1" x="66.04" y="71.12" smashed="yes" rot="R180">
+<attribute name="NAME" x="68.58" y="68.58" size="1.778" layer="95" rot="R180"/>
+</instance>
 </instances>
 <busses>
@@
 </segment>
 <segment>
-<wire x1="73.66" y1="68.58" x2="88.9" y2="68.58" width="0.1524" layer="91"/>
-<wire x1="88.9" y1="68.58" x2="88.9" y2="63.5" width="0.1524" layer="91"/>
+<wire x1="70.485" y1="71.12" x2="88.9" y2="71.12" width="0.1524" layer="91"/>
+<wire x1="88.9" y1="71.12" x2="88.9" y2="63.5" width="0.1524" layer="91"/>
 <pinref part="GND11" gate="1" pin="GND"/>
+<pinref part="U$2" gate="G$1" pin="V+/VCC"/>
 </segment>
 <segment>
@@
 <pinref part="K2" gate="1" pin="2"/>
 <wire x1="88.9" y1="76.2" x2="88.9" y2="73.66" width="0.1524" layer="91"/>
-<wire x1="88.9" y1="73.66" x2="73.66" y2="73.66" width="0.1524" layer="91"/>
+<wire x1="88.9" y1="73.66" x2="70.485" y2="73.66" width="0.1524" layer="91"/>
 <label x="73.66" y="73.66" size="1.778" layer="95"/>
 <pinref part="D4" gate="1" pin="A"/>
@@
 <wire x1="81.28" y1="76.2" x2="88.9" y2="76.2" width="0.1524" layer="91"/>
 <junction x="88.9" y="76.2"/>
-</segment>
-</net>
+<pinref part="U$2" gate="G$1" pin="GND/COM"/>
+</segment>
+</net>
